File: Dragon32.kicad_sch (KiCad schematic)
At the start: 77 parts, among them IC1 74HCT273, IC10 74HCT32, IC11 74LS123N, IC12 LM1889N, IC15 CD4053, IC2 MC6847, IC3 74HCT00, IC4 74HCT20, IC5 74HCT86, IC6 74HCT393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

Commit message: supplement power filtering
Parts:
- added FB1, FB2: FerriteBead_Small, Inductor_SMD:L_0805_2012Metric_Pad1.15x1.40mm_HandSolder, symbol Device:FerriteBead_Small
- added J3: YUV Output, Connector_PinHeader_2.54mm:PinHeader_1x05_P2.54mm_Vertical, symbol Connector:Conn_01x05_Pin
- added J4: S-Video Test, Connector_PinHeader_2.54mm:PinHeader_1x04_P2.54mm_Vertical, symbol Connector:Conn_01x04_Pin
- C1: value 100uF -> 10uF
- C19: footprint Capacitor_SMD:CP_Elec_6.3x5.8 -> Dragon:CP_Elec_10x10.5
- U2: value MCP6281 -> TS971; DigiKey (none) -> 497-8150-1-ND
Connections:
- net +5V: now also U2.5 (Vdd), FB1.1, FB2.2, J3.1 (Pin_1), J4.1 (Pin_1); no longer J1.1 (Pin_1), J2.2 (Pin_2), U2.2 (Vdd)
- net -5V: now also J2.3 (Pin_3), U2.2 (Vss); no longer U2.5 (Vss)
- net Chroma: now also J4.4 (Pin_4)
- net GND: now also J3.3 (Pin_3), J4.3 (Pin_3)
- net LUM: now also J3.2 (Pin_2)
- net MUX X: now also J4.2 (Pin_2)
- net phiA: now also J3.4 (Pin_4)
- net phiB: now also J3.5 (Pin_5)
- new net: FB2.1, J2.2 (Pin_2)
- new net: FB1.2, J1.1 (Pin_1)
- no-connect marks 50 -> 49

Commit message: refinement
Parts:
- added TP14: TestPoint_SyncPulse, TestPoint:TestPoint_Pad_D1.0mm, symbol Connector:TestPoint_Probe
Connections:
- net CHB: now also U2.3 (Vin+); no longer U2.4 (Vin-)
- net MUX Zinput: now also TP14.1
- net at C14.1, R12.1, R9.2: now also U2.4 (Vin-); no longer U2.3 (Vin+)
Other:
- moved on the sheet: C12, C14, R12, R9
