File: Dragon32.kicad_sch (KiCad schematic)
At the start: 64 parts, among them IC10 2318, IC11 MC14053, IC12 MC6847, IC13 74LS273N, IC14 74LS86AN, IC21 74LS123N, IC22 74LS00N, IC23 74ALS74N, IC27 74LS20N, IC28 74LS393N, IC29 74LS393N, IC3 74LS00N, IC30 74LS32N, IC32 74LS390, IC5 74LS86AN, IC6 74LS393N, IC7 74ALS74N, IC9 LM1889N, J1 Board interconnect, J2 Video Output, Y1 4.433619MHz

Commit message: fix missing css and fs signals
Parts:
- removed J1: Board interconnect, Connector_PinHeader_2.54mm:PinHeader_2x10_P2.54mm_Vertical, symbol Connector_Generic:Conn_02x10_Odd_Even
- added J1: Board Interconnect Male, Connector_PinHeader_2.54mm:PinHeader_2x11_P2.54mm_Vertical, symbol Connector_Generic:Conn_02x11_Odd_Even
- renumbered C36 to C1, C28 to C10, C24 to C11, C25 to C12, C49 to C13, C6 to C14, C8 to C15, C29 to C16, C9 to C17, C5 to C2, C34 to C3, C46 to C4, C47 to C5, C2 to C6, C3 to C8, C71 to C9, IC13 to IC1, IC30 to IC10, IC21 to IC11, IC9 to IC12, IC10 to IC13, IC11 to IC15, IC12 to IC2, IC22 to IC3, IC27 to IC4, IC14 to IC5, IC28 to IC6, IC23 to IC7, IC29 to IC8, IC32 to IC9, R4 to R1, R7 to R10, R6 to R11, R18 to R12, R11 to R13, R65 to R14, R67 to R15, R68 to R16, R10 to R17, R69 to R18, R76 to R19, R8 to R20, R9 to R21, R44 to R4, R35 to R6, R34 to R7, R33 to R8, R17 to R9, TR3 to TR1, TR4 to TR3
Connections:
- net +5V: now also J1.1 (Pin_1)
- net -5V: now also J1.2 (Pin_2)
- net CSS: now also J1.19 (Pin_19)
- net DA0: now also J1.6 (Pin_6)
- net DO0: now also J1.3 (Pin_3)
- net DO1: now also J1.5 (Pin_5)
- net DO2: now also J1.7 (Pin_7)
- net DO3: now also J1.9 (Pin_9)
- net DO4: now also J1.11 (Pin_11)
- net DO5: now also J1.13 (Pin_13)
- net DO6: now also J1.15 (Pin_15)
- net DO7: now also J1.17 (Pin_17)
- net GM0: now also J1.14 (Pin_14)
- net GM1: now also J1.12 (Pin_12)
- net GM2: now also J1.10 (Pin_10)
- net GND: now also J1.4 (Pin_4)
- net VCLK: now also J1.18 (Pin_18)
- net ~{A}/G: now also J1.20 (Pin_20)
- net ~{FS}: now also J1.22 (Pin_22)
- net ~{NHS}: now also J1.8 (Pin_8)
- net ~{RAS0}: now also J1.16 (Pin_16)

Commit message: partial conversion
Parts:
- C1: footprint Capacitor_THT:CP_Radial_D6.3mm_P2.50mm -> Capacitor_SMD:CP_Elec_6.3x5.8
- C10, C11: footprint Capacitor_THT:CP_Radial_D5.0mm_P2.50mm -> Capacitor_SMD:CP_Elec_5x5.8
- C12, C15, C6: footprint Capacitor_THT:C_Disc_D4.3mm_W1.9mm_P5.00mm -> Capacitor_SMD:C_0805_2012Metric_Pad1.18x1.45mm_HandSolder
- C13, C14, C17, C2, C3, C4, C5, C8, C9: footprint Capacitor_THT:C_Disc_D3.0mm_W2.0mm_P2.50mm -> Capacitor_SMD:C_0805_2012Metric_Pad1.18x1.45mm_HandSolder
- C16: footprint Capacitor_THT:CP_Radial_D5.0mm_P2.50mm -> Capacitor_SMD:CP_Elec_4x5.4
- IC1: value 74LS273N -> 74HCT273; footprint Package_DIP:DIP-20_W7.62mm -> Package_SO:TSSOP-20_4.4x6.5mm_P0.65mm
- IC10: value 74LS32N -> 74HCT32; footprint Package_DIP:DIP-14_W7.62mm -> Package_SO:SOIC-16_3.9x9.9mm_P1.27mm
- IC11: footprint Package_DIP:DIP-16_W7.62mm -> Package_SO:SOIC-16_3.9x9.9mm_P1.27mm
- IC15: value MC14053 -> CD4053; footprint Package_DIP:DIP-16_W7.62mm -> Package_SO:SOIC-16_3.9x9.9mm_P1.27mm
- IC3: value 74LS00N -> 74HCT00; footprint Package_DIP:DIP-14_W7.62mm -> Package_SO:SOIC-14_3.9x8.7mm_P1.27mm
- IC4: value 74LS20N -> 74HCT20; footprint Package_DIP:DIP-14_W7.62mm -> Package_SO:SOIC-14_3.9x8.7mm_P1.27mm
- IC5: value 74LS86AN -> 74HCT86; footprint Package_DIP:DIP-14_W7.62mm -> Package_SO:SOIC-14_3.9x8.7mm_P1.27mm
- IC6, IC8: value 74LS393N -> 74HCT393; footprint Package_DIP:DIP-14_W7.62mm -> Package_SO:SOIC-14_3.9x8.7mm_P1.27mm
- IC7: footprint Package_DIP:DIP-14_W7.62mm -> Package_SO:SOIC-14_3.9x8.7mm_P1.27mm
- IC9: value 74LS390 -> 74HCT390; footprint Package_DIP:DIP-16_W7.62mm -> Package_SO:SOIC-16_3.9x9.9mm_P1.27mm
- R1, R10, R11, R12, R13, R14, R15, R16, R17, R18, R19, R2, R20, R21, R3, R4, R5, R6, R7, R8, R9: footprint Resistor_THT:R_Axial_DIN0207_L6.3mm_D2.5mm_P2.54mm_Vertical -> Resistor_SMD:R_0805_2012Metric_Pad1.20x1.40mm_HandSolder

Commit message: complete tracing for fabrication
Parts:
- IC1: DigiKey 296-1657-5-ND -> 296-8409-1-ND
Changed lines of the file:
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@@
       (effects (font (size 1.27 1.27)) hide)
     )
-    (property "DigiKey" "296-1657-5-ND" (at 42.672 45.72 0)
+    (property "DigiKey" "296-8409-1-ND" (at 42.672 45.72 0)
       (effects (font (size 1.27 1.27)) hide)
     )

Commit message: update board
Parts:
- IC10: footprint Package_SO:SOIC-16_3.9x9.9mm_P1.27mm -> Package_SO:SOIC-14_3.9x8.7mm_P1.27mm
- IC6, IC8: DigiKey 296-1665-5-ND -> 296-14556-1-ND
Changed lines of the file:
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@@
       (effects (font (size 1.27 1.27)) hide)
     )
-    (property "DigiKey" "296-1665-5-ND" (at 85.471 247.777 0)
+    (property "DigiKey" "296-14556-1-ND" (at 85.471 247.777 0)
       (effects (font (size 1.27 1.27)) hide)
     )
@@
       (effects (font (size 1.27 1.27)) hide)
     )
-    (property "DigiKey" "296-1665-5-ND" (at 391.16 235.585 0)
+    (property "DigiKey" "296-14556-1-ND" (at 391.16 235.585 0)
       (effects (font (size 1.27 1.27)) hide)
     )
@@
       (effects (font (size 1.27 1.27)) hide)
     )
-    (property "DigiKey" "296-1665-5-ND" (at 344.932 152.908 0)
+    (property "DigiKey" "296-14556-1-ND" (at 344.932 152.908 0)
       (effects (font (size 1.27 1.27)) hide)
     )
@@
       (effects (font (size 1.27 1.27)))
     )
-    (property "Footprint" "Package_SO:SOIC-16_3.9x9.9mm_P1.27mm" (at 143.002 250.571 0)
+    (property "Footprint" "Package_SO:SOIC-14_3.9x8.7mm_P1.27mm" (at 143.002 250.571 0)
       (effects (font (size 1.27 1.27)) hide)
     )
@@
       (effects (font (size 1.27 1.27)))
     )
-    (property "Footprint" "Package_SO:SOIC-16_3.9x9.9mm_P1.27mm" (at 162.052 258.953 0)
+    (property "Footprint" "Package_SO:SOIC-14_3.9x8.7mm_P1.27mm" (at 162.052 258.953 0)
       (effects (font (size 1.27 1.27)) hide)
     )
@@
       (effects (font (size 1.27 1.27)) hide)
     )
-    (property "DigiKey" "296-1665-5-ND" (at 86.36 165.354 0)
+    (property "DigiKey" "296-14556-1-ND" (at 86.36 165.354 0)
       (effects (font (size 1.27 1.27)) hide)
     )
@@
       (effects (font (size 1.27 1.27)) (justify left))
     )
-    (property "Footprint" "Package_SO:SOIC-16_3.9x9.9mm_P1.27mm" (at 370.713 236.601 0)
+    (property "Footprint" "Package_SO:SOIC-14_3.9x8.7mm_P1.27mm" (at 370.713 236.601 0)
       (effects (font (size 1.27 1.27)) hide)
     )
@@
       (effects (font (size 1.27 1.27)))
     )
-    (property "Footprint" "Package_SO:SOIC-16_3.9x9.9mm_P1.27mm" (at 142.875 266.7 0)
+    (property "Footprint" "Package_SO:SOIC-14_3.9x8.7mm_P1.27mm" (at 142.875 266.7 0)
       (effects (font (size 1.27 1.27)) hide)
     )
@@
       (effects (font (size 1.27 1.27)) hide)
     )
-    (property "DigiKey" "296-1665-5-ND" (at 53.848 162.814 0)
+    (property "DigiKey" "296-14556-1-ND" (at 53.848 162.814 0)
       (effects (font (size 1.27 1.27)) hide)
     )
@@
       (effects (font (size 1.27 1.27)))
     )
-    (property "Footprint" "Package_SO:SOIC-16_3.9x9.9mm_P1.27mm" (at 313.944 240.284 0)
+    (property "Footprint" "Package_SO:SOIC-14_3.9x8.7mm_P1.27mm" (at 313.944 240.284 0)
       (effects (font (size 1.27 1.27)) hide)
     )
@@
       (effects (font (size 1.27 1.27)) hide)
     )
-    (property "DigiKey" "296-1665-5-ND" (at 112.522 255.397 0)
+    (property "DigiKey" "296-14556-1-ND" (at 112.522 255.397 0)
       (effects (font (size 1.27 1.27)) hide)
     )

Commit message: redesign smd approach
Parts:
- removed IC13: 2318, Package_DIP:DIP-8_W7.62mm, symbol vdg:SFC2318DC
- removed TR1, TR2: 2N2369, Package_TO_SOT_THT:TO-92_Inline_Wide, symbol Transistor_BJT:BC141
- removed TR3: BC212, Package_TO_SOT_THT:TO-92_Inline_Wide, symbol Transistor_BJT:2N3906
- added D1, D2: CD4148WT, PCM_Diode_SMD_AKL:D_0603_1608Metric, symbol PCM_Diode_AKL:CD4148WT
- added IC13: MCP6281T-E-OT, PCM_Package_TO_SOT_SMD_AKL:SOT-23-5, symbol PCM_Amplifier_Operational_AKL:MCP6281T-E-OT
- added TR1, TR2: MMBT4401, Package_TO_SOT_SMD:SOT-23-3, symbol PCM_Transistor_BJT_AKL:MMBT4401
- added TR3: BC857B, Package_TO_SOT_SMD:SOT-23-3, symbol PCM_Transistor_BJT_AKL:BC857B
- added Y2: CXO_DIP14, Oscillator:Oscillator_DIP-14, symbol Oscillator:CXO_DIP14
- added Y3: ASCO, Oscillator:Oscillator_SMD_Abracon_ASV-4Pin_7.0x5.1mm_HandSoldering, symbol Oscillator:ASCO
- added Y4: CXO_DIP8, Oscillator:Oscillator_DIP-8, symbol Oscillator:CXO_DIP8
- C1: LCSC (none) -> C7469933
- C10: footprint Capacitor_SMD:CP_Elec_5x5.8 -> Capacitor_Tantalum_SMD:CP_EIA-3528-15_AVX-H; DigiKey 478-8984-1-ND -> 478-3886-1-ND; LCSC (none) -> C140403
- C11: footprint Capacitor_SMD:CP_Elec_5x5.8 -> Capacitor_Tantalum_SMD:CP_EIA-3528-15_AVX-H; DigiKey 478-8984-1-ND -> 478-11463-1-ND; LCSC (none) -> C136751
- C12, C15: LCSC (none) -> C1710
- C13, C17: LCSC (none) -> C1804
- C14: footprint Capacitor_SMD:C_0805_2012Metric_Pad1.18x1.45mm_HandSolder -> Capacitor_SMD:C_0603_1608Metric; LCSC (none) -> C1669
- C16: LCSC (none) -> C3348
- C2, C8: footprint Capacitor_SMD:C_0805_2012Metric_Pad1.18x1.45mm_HandSolder -> Capacitor_SMD:C_0603_1608Metric; DigiKey BC1007CT-ND -> (none); LCSC (none) -> C1663
- C3: footprint Capacitor_SMD:C_0805_2012Metric_Pad1.18x1.45mm_HandSolder -> Capacitor_SMD:C_0603_1608Metric; DigiKey BC1045CT-ND -> (none); LCSC (none) -> C1664
- C4, C9: LCSC (none) -> C113826
- C5: LCSC (none) -> C1790
- C6: LCSC (none) -> C28233
- IC1: LCSC (none) -> C484754
- IC10: LCSC (none) -> C5985
- IC11: LCSC (none) -> C1522784
- IC12: LCSC (none) -> C72116
- IC15: footprint Package_SO:SOIC-16_3.9x9.9mm_P1.27mm -> Package_SO:SOIC-16_4.55x10.3mm_P1.27mm; LCSC (none) -> C6742
- IC2: LCSC (none) -> C72123
- IC3: LCSC (none) -> C6764
- IC4: LCSC (none) -> C5975
- IC5: LCSC (none) -> C527451
- IC6, IC8: LCSC (none) -> C547642
- IC7: LCSC (none) -> C897306
- IC9: LCSC (none) -> C1548010
- J1, J2: now left out of the parts list
- R1: LCSC (none) -> C26010
- R10: LCSC (none) -> C17560
- R11, R2, R5: LCSC (none) -> C17513
- R12, R9: LCSC (none) -> C17414
- R13, R14, R17: LCSC (none) -> C17530
- R15: LCSC (none) -> C17379
- R16, R3: LCSC (none) -> C4382
- R18: LCSC (none) -> C17630
- R19: LCSC (none) -> C17415
- R20, R21: LCSC (none) -> C17590
- R4: LCSC (none) -> C17953
- R6: LCSC (none) -> C17444
- R7: LCSC (none) -> C17828
- R8: LCSC (none) -> C17398
- RV1: footprint Potentiometer_THT:Potentiometer_Bourns_3386X_Horizontal -> Potentiometer_SMD:Potentiometer_Bourns_3314J_Vertical; DigiKey 3386H-103LF-ND -> (none); LCSC (none) -> C36376
Connections:
- net +5V: now also IC13.5 (V+), TR2.3 (C), Y2.14 (Vcc), Y3.4 (VDD), Y4.8 (Vcc)
- net -5V: now also J2.3 (Pin_3), IC13.2 (V-), TR3.3 (C); no longer J1.2 (Pin_2)
- net CHB: now also IC13.3 (+)
- net ChrOSC: now also Y2.8 (OUT), Y3.3 (OUT), Y4.5 (OUT)
- net GND: now also D2.1 (K), TR1.2 (E), Y2.7 (GND), Y3.2 (GND), Y4.4 (GND); no longer RV1.3
- net at R17.1, R18.2, R19.2: now also TR2.2 (E), TR3.1 (B)
- net at R11.2, R13.2, R14.1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: now also TR1.1 (B)
- net at C14.1, R12.1, R9.2: now also IC13.4 (-)
- net at C14.2, IC15.5 (Z0), R12.2: now also IC13.1
- net at C17.2, R16.1: now also TR1.3 (C), TR2.1 (B)
- net at R21.1: now also TR3.2 (E)
- new net: D1.1 (K), D2.2 (A)
- new net: D1.2 (A), RV1.3
Other:
- moved on the sheet: C2, C6, R2, R5
